Commit message: Initial commit of xarm_ros2 workspace

File: xarm_moveit_config/srdf/_lite6_macro.srdf.xacro (robot description, xacro)
@@ -36,10 +36,10 @@
     <!-- GROUP STATES, Purpose, Define a named state for a particular group, in terms of joint values. This is useful to define states like 'folded arms' -->
     <group_state name="home" group="${prefix}lite6">
-      <joint name="${prefix}joint1" value="0" />
-      <joint name="${prefix}joint2" value="0" />
-      <joint name="${prefix}joint3" value="0" />
-      <joint name="${prefix}joint4" value="0" />
-      <joint name="${prefix}joint5" value="0" />
-      <joint name="${prefix}joint6" value="0" />
+      <joint name="${prefix}joint1" value="0.08166910523670001" />
+      <joint name="${prefix}joint2" value="0.4753780559040486" />
+      <joint name="${prefix}joint3" value="1.4820387149899972" />
+      <joint name="${prefix}joint4" value="-0.14591265543817933" />
+      <joint name="${prefix}joint5" value="0.3513251124160188" />
+      <joint name="${prefix}joint6" value="0.201567773671691" />
     </group_state>
     <!-- gripper -->
